Commit message: Corrections to the WHEEL_SEPERAION

File: robot_bringup/config/robot.urdf (robot description, URDF)
Before this commit: robot tierbee_robot, 6 links, 5 joints
Joints:
- joint left_wheel_joint: origin xyz=0.0 0.112 -0.019 rpy=0 0 0 -> xyz=0.0 0.085 -0.019 rpy=0 0 0
- joint right_wheel_joint: origin xyz=0.0 -0.112 -0.019 rpy=0 0 0 -> xyz=0.0 -0.085 -0.019 rpy=0 0 0
